File: hardware/ps2plus.sch (KiCad schematic (older format))
At the start: 39 parts, among them J1 Conn_01x06_Female, Q1 2N7000, U1 PIC16F18876-I_PT

Commit message: Updated pcb design, still not completely optimal
Parts:
- J1: footprint Connector_PinHeader_2.54mm:PinHeader_1x06_P2.54mm_Horizontal -> Connector_PinHeader_2.54mm:PinHeader_1x06_P2.54mm_Vertical
- Q1: footprint Package_TO_SOT_THT:TO-92_Inline -> Package_TO_SOT_SMD:SOT-23
- TP12: renamed from TP28; value DDOWN -> DD
- TP15: renamed from TP31; value CS -> ATN
- TP3: value 8.5V -> RMB
- renumbered MOSI1 to CMD1, MISO1 to DAT1, DLEFT1 to DL1, DRIGHT1 to DR1, DUP to DU1, TP24 to TP10, TP25 to TP11, TP29 to TP13, TP30 to TP14, TP32 to TP16, TP14 to TP4, TP15 to TP5, TP16 to TP6, TP17 to TP7, TP20 to TP8, TP22 to TP9
Changed lines of the file:
@@
 U 1 1 5D46DA1F
 P 6900 2700
-F 0 "LX1" V 6900 3200 50  0000 L CNN
-F 1 "TP26" V 6900 2900 50  0000 L CNN
+F 0 "LX1" V 6900 2900 50  0000 L CNN
+F 1 "TP26" V 6900 3200 50  0000 L CNN
 F 2 "TestPoint:TestPoint_Pad_2.0x2.0mm" H 7100 2700 50  0001 C CNN
 F 3 "~" H 7100 2700 50  0001 C CNN
@@
 $EndComp
 $Comp
-L Connector:TestPoint DUP
+L Connector:TestPoint DU1
 U 1 1 5D46E7EF
 P 6900 2800
-F 0 "DUP" V 6900 3000 50  0000 L CNN
+F 0 "DU1" V 6900 3000 50  0000 L CNN
 F 1 "TP27" V 6900 3300 50  0000 L CNN
 F 2 "TestPoint:TestPoint_Pad_2.0x2.0mm" H 7100 2800 50  0001 C CNN
@@
 $EndComp
 $Comp
-L Connector:TestPoint TP28
+L Connector:TestPoint TP12
 U 1 1 5D46E821
 P 6900 2900
-F 0 "TP28" V 6900 3400 50  0000 L CNN
-F 1 "DDOWN" V 6900 3100 50  0000 L CNN
+F 0 "TP12" V 6900 3400 50  0000 L CNN
+F 1 "DD" V 6900 3100 50  0000 L CNN
 F 2 "TestPoint:TestPoint_Pad_2.0x2.0mm" H 7100 2900 50  0001 C CNN
 F 3 "~" H 7100 2900 50  0001 C CNN
@@
 $EndComp
 $Comp
-L Connector:TestPoint TP29
+L Connector:TestPoint TP13
 U 1 1 5D46E9F4
 P 6900 3000
-F 0 "TP29" V 6900 3500 50  0000 L CNN
+F 0 "TP13" V 6900 3500 50  0000 L CNN
 F 1 "GND" V 6900 3200 50  0000 L CNN
 F 2 "TestPoint:TestPoint_Pad_2.0x2.0mm" H 7100 3000 50  0001 C CNN
@@
 $EndComp
 $Comp
-L Connector:TestPoint TP30
+L Connector:TestPoint TP14
 U 1 1 5D46EC3A
 P 6900 3100
-F 0 "TP30" V 6900 3600 50  0000 L CNN
+F 0 "TP14" V 6900 3600 50  0000 L CNN
 F 1 "3.3V" V 6900 3300 50  0000 L CNN
 F 2 "TestPoint:TestPoint_Pad_2.0x2.0mm" H 7100 3100 50  0001 C CNN
@@
 $EndComp
 $Comp
-L Connector:TestPoint TP31
+L Connector:TestPoint TP15
 U 1 1 5D46EFE6
 P 6900 3500
-F 0 "TP31" V 6900 4000 50  0000 L CNN
-F 1 "CS" V 6900 3700 50  0000 L CNN
+F 0 "TP15" V 6900 4000 50  0000 L CNN
+F 1 "ATN" V 6900 3700 50  0000 L CNN
 F 2 "TestPoint:TestPoint_Pad_2.0x2.0mm" H 7100 3500 50  0001 C CNN
 F 3 "~" H 7100 3500 50  0001 C CNN
@@
 $EndComp
 $Comp
-L Connector:TestPoint TP32
+L Connector:TestPoint TP16
 U 1 1 5D46F0E7
 P 6900 3600
-F 0 "TP32" V 6900 4100 50  0000 L CNN
+F 0 "TP16" V 6900 4100 50  0000 L CNN
 F 1 "ACK" V 6900 3800 50  0000 L CNN
 F 2 "TestPoint:TestPoint_Pad_2.0x2.0mm" H 7100 3600 50  0001 C CNN
@@
 $EndComp
 $Comp
-L Connector:TestPoint TP14
+L Connector:TestPoint TP4
 U 1 1 5D471BC4
 P 5350 4250
-F 0 "TP14" H 5450 4750 50  0000 R CNN
+F 0 "TP4" H 5450 4750 50  0000 R CNN
 F 1 "R1" H 5400 4550 50  0000 R CNN
 F 2 "TestPoint:TestPoint_Pad_2.0x2.0mm" H 5550 4250 50  0001 C CNN
@@
 $EndComp
 $Comp
-L Connector:TestPoint TP15
+L Connector:TestPoint TP5
 U 1 1 5D471FCB
 P 5450 4250
-F 0 "TP15" H 5500 4650 50  0000 R CNN
+F 0 "TP5" H 5500 4650 50  0000 R CNN
 F 1 "R2" H 5500 4450 50  0000 R CNN
 F 2 "TestPoint:TestPoint_Pad_2.0x2.0mm" H 5650 4250 50  0001 C CNN
@@
 $EndComp
 $Comp
-L Connector:TestPoint TP16
+L Connector:TestPoint TP6
 U 1 1 5D472132
 P 5550 4250
-F 0 "TP16" H 5550 4750 50  0000 R CNN
+F 0 "TP6" H 5550 4750 50  0000 R CNN
 F 1 "SL" H 5600 4550 50  0000 R CNN
 F 2 "TestPoint:TestPoint_Pad_2.0x2.0mm" H 5750 4250 50  0001 C CNN
@@
 $EndComp
 $Comp
-L Connector:TestPoint TP17
+L Connector:TestPoint TP7
 U 1 1 5D472186
 P 5650 4250
-F 0 "TP17" H 5600 4650 50  0000 R CNN
+F 0 "TP7" H 5600 4650 50  0000 R CNN
 F 1 "ST" H 5700 4450 50  0000 R CNN
 F 2 "TestPoint:TestPoint_Pad_2.0x2.0mm" H 5850 4250 50  0001 C CNN
@@
 $EndComp
 $Comp
-L Connector:TestPoint TP20
+L Connector:TestPoint TP8
 U 1 1 5D47235B
 P 5850 4250
-F 0 "TP20" H 5850 4750 50  0000 R CNN
+F 0 "TP8" H 5850 4750 50  0000 R CNN
 F 1 "SQ" H 5900 4550 50  0000 R CNN
 F 2 "TestPoint:TestPoint_Pad_2.0x2.0mm" H 6050 4250 50  0001 C CNN
@@
 $EndComp
 $Comp
-L Connector:TestPoint TP22
+L Connector:TestPoint TP9
 U 1 1 5D472448
 P 5950 4250
-F 0 "TP22" H 5900 4650 50  0000 R CNN
+F 0 "TP9" H 5900 4650 50  0000 R CNN
 F 1 "TRI" H 6000 4450 50  0000 R CNN
 F 2 "TestPoint:TestPoint_Pad_2.0x2.0mm" H 6150 4250 50  0001 C CNN
@@
 $EndComp
 $Comp
-L Connector:TestPoint TP24
+L Connector:TestPoint TP10
 U 1 1 5D4724F2
 P 6050 4250
-F 0 "TP24" H 5950 4750 50  0000 R CNN
+F 0 "TP10" H 5950 4750 50  0000 R CNN
 F 1 "X" H 6050 4550 50  0000 R CNN
 F 2 "TestPoint:TestPoint_Pad_2.0x2.0mm" H 6250 4250 50  0001 C CNN
@@
 $EndComp
 $Comp
-L Connector:TestPoint TP25
+L Connector:TestPoint TP11
 U 1 1 5D472736
 P 6150 4250
-F 0 "TP25" H 6000 4650 50  0000 R CNN
+F 0 "TP11" H 6000 4650 50  0000 R CNN
 F 1 "CIR" H 6150 4450 50  0000 R CNN
 F 2 "TestPoint:TestPoint_Pad_2.0x2.0mm" H 6350 4250 50  0001 C CNN
@@
 $EndComp
 $Comp
-L Connector:TestPoint DLEFT1
+L Connector:TestPoint DL1
 U 1 1 5D47166F
 P 4500 3300
-F 0 "DLEFT1" V 4500 3900 50  0000 C CNN
+F 0 "DL1" V 4500 3900 50  0000 C CNN
 F 1 "TP7" V 4500 3550 50  0000 C CNN
 F 2 "TestPoint:TestPoint_Pad_2.0x2.0mm" H 4700 3300 50  0001 C CNN
@@
 $EndComp
 $Comp
-L Connector:TestPoint DRIGHT1
+L Connector:TestPoint DR1
 U 1 1 5D471797
 P 4500 3400
-F 0 "DRIGHT1" V 4500 4000 50  0000 C CNN
+F 0 "DR1" V 4500 4000 50  0000 C CNN
 F 1 "TP8" V 4500 3650 50  0000 C CNN
 F 2 "TestPoint:TestPoint_Pad_2.0x2.0mm" H 4700 3400 50  0001 C CNN
@@
 U 1 1 5D471A04
 P 4500 3600
-F 0 "L2" V 4500 4250 50  0000 C CNN
+F 0 "L2" V 4500 4200 50  0000 C CNN
 F 1 "TP10" V 4500 3850 50  0000 C CNN
 F 2 "TestPoint:TestPoint_Pad_2.0x2.0mm" H 4700 3600 50  0001 C CNN
@@
 U 1 1 5D4718BD
 P 4500 3500
-F 0 "L1" V 4500 4150 50  0000 C CNN
+F 0 "L1" V 4500 4100 50  0000 C CNN
 F 1 "TP9" V 4500 3750 50  0000 C CNN
 F 2 "TestPoint:TestPoint_Pad_2.0x2.0mm" H 4700 3500 50  0001 C CNN
@@
 F 0 "Q1" H 1806 2604 50  0000 L CNN
 F 1 "2N7000" H 1806 2695 50  0000 L CNN
-F 2 "Package_TO_SOT_THT:TO-92_Inline" H 1800 2575 50  0001 L CIN
+F 2 "Package_TO_SOT_SMD:SOT-23" H 1800 2575 50  0001 L CIN
 F 3 "https://www.fairchildsemi.com/datasheets/2N/2N7000.pdf" H 1600 2650 50  0001 L CNN
 	1    1600 2650
@@
 P 1500 3750
 F 0 "TP3" H 1442 3776 50  0000 R CNN
-F 1 "8.5V" H 1442 3867 50  0000 R CNN
+F 1 "RMB" H 1442 3867 50  0000 R CNN
 F 2 "TestPoint:TestPoint_Pad_2.0x2.0mm" H 1700 3750 50  0001 C CNN
 F 3 "~" H 1700 3750 50  0001 C CNN
@@
 Connection ~ 6650 3100
 $Comp
-L power:+3.3V #PWR0101
+L power:+3.3V #PWR06
 U 1 1 5D4DEC95
 P 7850 3100
-F 0 "#PWR0101" H 7850 2950 50  0001 C CNN
+F 0 "#PWR06" H 7850 2950 50  0001 C CNN
 F 1 "+3.3V" V 7865 3228 50  0000 L CNN
 F 2 "" H 7850 3100 50  0001 C CNN
@@
 $EndComp
 $Comp
-L power:+3.3V #PWR0102
+L power:+3.3V #PWR04
 U 1 1 5D4DF831
 P 3650 3200
-F 0 "#PWR0102" H 3650 3050 50  0001 C CNN
+F 0 "#PWR04" H 3650 3050 50  0001 C CNN
 F 1 "+3.3V" V 3665 3328 50  0000 L CNN
 F 2 "" H 3650 3200 50  0001 C CNN
@@
 $EndComp
 $Comp
-L power:GNDREF #PWR0103
+L power:GNDREF #PWR05
 U 1 1 5D4E0E22
 P 7850 3000
-F 0 "#PWR0103" H 7850 2750 50  0001 C CNN
+F 0 "#PWR05" H 7850 2750 50  0001 C CNN
 F 1 "GNDREF" V 7855 2872 50  0000 R CNN
 F 2 "" H 7850 3000 50  0001 C CNN
@@
 $EndComp
 $Comp
-L power:GNDREF #PWR0104
+L power:GNDREF #PWR03
 U 1 1 5D4E1FF5
 P 3650 3100
-F 0 "#PWR0104" H 3650 2850 50  0001 C CNN
+F 0 "#PWR03" H 3650 2850 50  0001 C CNN
 F 1 "GNDREF" V 3655 2972 50  0000 R CNN
 F 2 "" H 3650 3100 50  0001 C CNN
@@
 Connection ~ 4500 3200
 $Comp
-L power:PWR_FLAG #FLG0101
+L power:PWR_FLAG #FLG02
 U 1 1 5D4EA98D
 P 7750 3200
-F 0 "#FLG0101" H 7750 3275 50  0001 C CNN
+F 0 "#FLG02" H 7750 3275 50  0001 C CNN
 F 1 "PWR_FLAG" H 7750 3373 50  0000 C CNN
 F 2 "" H 7750 3200 50  0001 C CNN
@@
 $EndComp
 $Comp
-L power:PWR_FLAG #FLG0102
+L power:PWR_FLAG #FLG01
 U 1 1 5D4EB44C
 P 7750 2900
-F 0 "#FLG0102" H 7750 2975 50  0001 C CNN
+F 0 "#FLG01" H 7750 2975 50  0001 C CNN
 F 1 "PWR_FLAG" H 7850 3050 50  0000 C CNN
 F 2 "" H 7750 2900 50  0001 C CNN
@@
 F 0 "J1" V 5646 5548 50  0000 L CNN
 F 1 "Conn_01x06_Female" V 5737 5548 50  0000 L CNN
-F 2 "Connector_PinHeader_2.54mm:PinHeader_1x06_P2.54mm_Horizontal" H 5800 5300 50  0001 C CNN
+F 2 "Connector_PinHeader_2.54mm:PinHeader_1x06_P2.54mm_Vertical" H 5800 5300 50  0001 C CNN
 F 3 "~" H 5800 5300 50  0001 C CNN
 	1    5800 5300
@@
 $EndComp
 $Comp
-L Connector:TestPoint MOSI1
+L Connector:TestPoint CMD1
 U 1 1 5D470360
 P 5350 1950
-F 0 "MOSI1" H 5350 2250 50  0000 L CNN
+F 0 "CMD1" H 5350 2250 50  0000 L CNN
 F 1 "TP13" H 5400 2450 50  0000 L CNN
 F 2 "TestPoint:TestPoint_Pad_2.0x2.0mm" H 5550 1950 50  0001 C CNN
@@
 $EndComp
 $Comp
-L Connector:TestPoint MISO1
+L Connector:TestPoint DAT1
 U 1 1 5D4704A8
 P 5250 1950
-F 0 "MISO1" H 5150 2150 50  0000 L CNN
+F 0 "DAT1" H 5150 2150 50  0000 L CNN
 F 1 "TP12" H 5200 2350 50  0000 L CNN
 F 2 "TestPoint:TestPoint_Pad_2.0x2.0mm" H 5450 1950 50  0001 C CNN
